Commit message: Changes to description

File: rover_description/robots/rover.urdf.xacro (robot description, xacro)
@@ -165,4 +165,8 @@
         <origin xyz="0.17 0 0.005" rpy="0 0 0"/>
     </xacro:sensor_hokuyo>
+    <xacro:include filename="$(find ros2_livox_simulation)/urdf/mid360.xacro"/>
+<xacro:mid360 parent="base_link" name="livox_lidar" topic="/livox/lidar">
+  <origin xyz="0.3 0 0.5" rpy="0 3.14 0" />
+</xacro:mid360>
     <xacro:sensor_imu prefix="imu" parent="base_link">
         <!-- <origin xyz="-0.32 0 0.05" rpy="0 0.5 0"/> -->
@@ -170,5 +174,5 @@
     </xacro:sensor_imu>
     <xacro:sensor_asus_xtion prefix="camera" parent="base_link">
-        <origin xyz="0.215 0 0.065" rpy="0 0.4 0"/>
+        <origin xyz="0.215 0 0.065" rpy="0 0 0"/>
         <!-- <origin xyz="0.212 0 0.065" rpy="0 0 0"/> -->
     </xacro:sensor_asus_xtion>

File: rover_description/urdf/materials.xacro (robot description, xacro)
@@ -18,5 +18,5 @@
 # SOFTWARE. -->
 <robot name="materials" xmlns:xacro="http://www.ros.org/wiki/xacro">
-    <material name="red">
+   <material name="red">
         <color rgba="0.8 0 0 1"/>
     </material>

File: rover_description/urdf/sensors/asus_xtion.urdf.xacro (robot description, xacro)
@@ -21,8 +21,8 @@
     <xacro:property name="math_pi_over_2" value="1.5707963267948966" />
     <joint name="${prefix}_joint" type="fixed">
-      <axis xyz="1 0 0"/>
-      <xacro:insert_block name="origin"/>
-      <parent link="${parent}"/>
-      <child link="${prefix}_link"/>
+        <axis xyz="1 0 0"/>
+        <xacro:insert_block name="origin"/>
+        <parent link="${parent}"/>
+        <child link="${prefix}_link"/>
     </joint>
     <link name="${prefix}_link">
@@ -76,5 +76,5 @@
             <far>8.0</far>
           </clip>
-          <distortion>
+	        <distortion>
             <k1>0.00000001</k1>
             <k2>0.00000001</k2>
@@ -137,5 +137,5 @@
                 </publisher>
               </topic>
-              <topic name="/camera/depth/image_raw/theora">
+             <topic name="/camera/depth/image_raw/theora">
                 <publisher>
                   <reliability>best_effort</reliability>

File: rover_description/urdf/sensors/hokuyo.urdf.xacro (robot description, xacro)
@@ -34,5 +34,5 @@
         <origin xyz="0 0 -0.05" rpy="0 0 0"/>
         <geometry>
-          <mesh filename="package://rover_description/meshes/sensors/hokuyo/hokuyo_ust_20lx.dae"/>
+            <mesh filename="package://rover_description/meshes/sensors/hokuyo/hokuyo_ust_20lx.dae"/>
         </geometry>
       </visual>
@@ -44,5 +44,5 @@
     </link>
     <gazebo reference="${prefix}_base_link">
-      <material>Gazebo/DarkGrey</material>
+        <material>Gazebo/DarkGrey</material>
     </gazebo>
     <link name="${prefix}_link">
@@ -54,43 +54,43 @@
     </joint>
     <gazebo reference="${prefix}_link">
-      <sensor type="gpu_ray" name="hokuyo_sensor">
-        <pose>0 0 0 0 0 0</pose>
-        <visualize>true</visualize>
-        <update_rate>50</update_rate>
-        <ray>
-          <scan>
-            <horizontal>
-              <samples>30</samples>
-              <resolution>1</resolution>
-              <min_angle>${min_angle}</min_angle>
-              <max_angle>${max_angle}</max_angle>
-            </horizontal>
-          </scan>
-          <range>
-            <min>0.06</min>
-            <max>5.0</max>
-            <resolution>0.004359297</resolution>
-          </range>
-          <noise>
-            <type>gaussian</type>
-            <mean>0.0</mean>
-            <stddev>0.01</stddev>
-          </noise>
-        </ray>
-        <plugin name="${prefix}_controller" filename="libgazebo_ros_ray_sensor.so">
-          <ros>
-            <remapping>~/out:=scan</remapping>
-            <qos>
-              <topic name="scan">
-                <publisher>
-                  <reliability>best_effort</reliability>
-                </publisher>
-              </topic>
-            </qos>
-          </ros>
-          <output_type>sensor_msgs/LaserScan</output_type>
-          <frame_name>${prefix}_link</frame_name>
-        </plugin>
-      </sensor>
+            <sensor type="gpu_ray" name="hokuyo_sensor">
+                <pose>0 0 0 0 0 0</pose>
+                <visualize>true</visualize>
+                <update_rate>50</update_rate>
+                <ray>
+                    <scan>
+                        <horizontal>
+                            <samples>30</samples>
+                            <resolution>1</resolution>
+                            <min_angle>${min_angle}</min_angle>
+                            <max_angle>${max_angle}</max_angle>
+                        </horizontal>
+                    </scan>
+                    <range>
+                        <min>0.06</min>
+                        <max>5.0</max>
+                        <resolution>0.004359297</resolution>
+                    </range>
+                    <noise>
+                        <type>gaussian</type>
+                        <mean>0.0</mean>
+                        <stddev>0.01</stddev>
+                    </noise>
+                </ray>
+                <plugin name="${prefix}_controller" filename="libgazebo_ros_ray_sensor.so">
+                  <ros>
+                    <remapping>~/out:=scan</remapping>
+                    <qos>
+                      <topic name="scan">
+                        <publisher>
+                          <reliability>best_effort</reliability>
+                        </publisher>
+                      </topic>
+                    </qos>
+                  </ros>
+                  <output_type>sensor_msgs/LaserScan</output_type>
+                  <frame_name>${prefix}_link</frame_name>
+                </plugin>
+            </sensor>
     </gazebo>
   </xacro:macro>

File: rover_description/urdf/sensors/imu.urdf.xacro (robot description, xacro)
@@ -20,8 +20,8 @@
   <xacro:macro name="sensor_imu" params="prefix parent *origin">
     <joint name="${prefix}_joint" type="fixed">
-      <axis xyz="1 0 0"/>
-      <xacro:insert_block name="origin"/>
-      <parent link="${parent}"/>
-      <child link="${prefix}_link"/>
+        <axis xyz="1 0 0"/>
+        <xacro:insert_block name="origin"/>
+        <parent link="${parent}"/>
+        <child link="${prefix}_link"/>
     </joint>
     <link name="${prefix}_link">
@@ -46,5 +46,5 @@
     </link>
     <gazebo reference="${prefix}_link">
-      <material>Gazebo/Blue</material>
+        <material>Gazebo/Blue</material>
     </gazebo>
     <gazebo reference="${prefix}_link">

File: rover_description/urdf/wheels/wheel.urdf.xacro (robot description, xacro)
@@ -46,9 +46,10 @@
         <gazebo reference="${lon_label}_${lat_label}_wheel_link">
             <material>Gazebo/DarkGray</material>
-            <mu1>1.0</mu1>
-            <mu2>1.0</mu2>
-            <kp>10000000</kp>
-            <kd>1.0</kd>
-            <fdir1 value="1 0 0"/>
+			<mu1 value="100.0"/>
+			<mu2 value="100.0"/>
+			<kp value="10000000.0" />
+			<kd value="1.0" />
+			<fdir1 value="1 0 0"/>
+            <turnGravityOff>false</turnGravityOff>
         </gazebo>
     </xacro:macro>

Commit message: camera added not working CHECK

File: rover_description/robots/rover.urdf.xacro (robot description, xacro)
@@ -177,4 +177,8 @@
         <!-- <origin xyz="0.212 0 0.065" rpy="0 0 0"/> -->
     </xacro:sensor_asus_xtion>
+    <xacro:sensor_asus_xtion2 prefix="camera" parent="base_link">
+        <origin xyz="0.215 0 1" rpy="0 1.57 0"/>
+        <!-- <origin xyz="0.212 0 0.065" rpy="0 0 0"/> -->
+    </xacro:sensor_asus_xtion2>
     <!-- wheels -->
     <xacro:corner_link lon_label="front" lat_label="left" reflect="1"/>

File: rover_description/urdf/sensors/all_sensors.urdf.xacro (robot description, xacro)
@@ -24,3 +24,4 @@
   <!-- Hokuyo -->
   <xacro:include filename="$(find rover_description)/urdf/sensors/asus_xtion.urdf.xacro" />
+  <xacro:include filename="$(find rover_description)/urdf/sensors/asus_xtion2.urdf.xacro" />
 </robot>

Commit message: added camera omn top

File: rover_description/robots/rover.urdf.xacro (robot description, xacro)
@@ -177,6 +177,6 @@
         <!-- <origin xyz="0.212 0 0.065" rpy="0 0 0"/> -->
     </xacro:sensor_asus_xtion>
-    <xacro:sensor_asus_xtion2 prefix="camera" parent="base_link">
-        <origin xyz="0.215 0 1" rpy="0 1.57 0"/>
+    <xacro:sensor_asus_xtion2 prefix="camera2" parent="base_link">
+        <origin xyz="0.215 0 5" rpy="0 1.57 0"/>
         <!-- <origin xyz="0.212 0 0.065" rpy="0 0 0"/> -->
     </xacro:sensor_asus_xtion2>

File: rover_description/urdf/sensors/asus_xtion2.urdf.xacro (robot description, xacro)
@@ -47,10 +47,10 @@
       </inertial>
     </link>
-    <joint name="camera_frame_joint" type="fixed">
+    <joint name="camera2_frame_joint" type="fixed">
       <origin xyz="0 0 0" rpy="-${math_pi_over_2} 0 -${math_pi_over_2}" />
       <parent link="${prefix}_link" />
-      <child link="camera_frame" />
+      <child link="camera2_frame" />
     </joint>
-    <link name="camera_frame">
+    <link name="camera2_frame">
       <inertial>
         <mass value="0.001" />
@@ -62,5 +62,5 @@
     </link>
     <gazebo reference="${prefix}_link">
-      <sensor name="camera" type="depth">
+      <sensor name="camera2" type="depth">
         <visualize>true</visualize>
         <update_rate>30</update_rate>
@@ -84,58 +84,58 @@
           </distortion>
         </camera>
-        <plugin name="depth_camera_controller" filename="libgazebo_ros_camera.so">
+        <plugin name="depth_camera2_controller" filename="libgazebo_ros_camera.so">
           <ros>
             <qos>
-              <topic name="/camera/camera_info">
+              <topic name="/camera2/camera_info">
                 <publisher>
                   <reliability>best_effort</reliability>
                 </publisher>
               </topic>
-              <topic name="/camera/image_raw">
+              <topic name="/camera2/image_raw">
                 <publisher>
                   <reliability>best_effort</reliability>
                 </publisher>
               </topic>
-              <topic name="/camera/image_raw/compressed">
+              <topic name="/camera2/image_raw/compressed">
                 <publisher>
                   <reliability>best_effort</reliability>
                 </publisher>
               </topic>
-              <topic name="/camera/image_raw/compressedDepth">
+              <topic name="/camera2/image_raw/compressedDepth">
                 <publisher>
                   <reliability>best_effort</reliability>
                 </publisher>
               </topic>
-              <topic name="/camera/image_raw/theora">
+              <topic name="/camera2/image_raw/theora">
                 <publisher>
                   <reliability>best_effort</reliability>
                 </publisher>
               </topic>
-              <topic name="/camera/points">
+              <topic name="/camera2/points">
                 <publisher>
                   <reliability>best_effort</reliability>
                 </publisher>
               </topic>
-              <topic name="/camera/depth/camera_info">
+              <topic name="/camera2/depth/camera_info">
                 <publisher>
                   <reliability>best_effort</reliability>
                 </publisher>
               </topic>
-              <topic name="/camera/depth/image_raw">
+              <topic name="/camera2/depth/image_raw">
                 <publisher>
                   <reliability>best_effort</reliability>
                 </publisher>
               </topic>
-              <topic name="/camera/depth/image_raw/compressed">
+              <topic name="/camera2/depth/image_raw/compressed">
                 <publisher>
                   <reliability>best_effort</reliability>
                 </publisher>
               </topic>
-              <topic name="/camera/depth/image_raw/compressedDepth">
+              <topic name="/camera2/depth/image_raw/compressedDepth">
                 <publisher>
                   <reliability>best_effort</reliability>
                 </publisher>
               </topic>
-             <topic name="/camera/depth/image_raw/theora">
+             <topic name="/camera2/depth/image_raw/theora">
                 <publisher>
                   <reliability>best_effort</reliability>
@@ -144,5 +144,5 @@
             </qos>
           </ros>
-          <frame_name>camera_frame</frame_name>
+          <frame_name>camera2_frame</frame_name>
           <min_depth>0.3</min_depth>
           <max_depth>8.0</max_depth>

Commit message: Lidar working in all worlds

File: rover_description/robots/rover.urdf.xacro (robot description, xacro)
@@ -25,4 +25,5 @@
             <joint_name>left_bogie_joint</joint_name>
             <joint_name>right_bogie_joint</joint_name>
+            <joint_name>livox_lidar_joint</joint_name>
             <joint_name>diff_brace_joint</joint_name>
             <joint_name>back_left_turnbuckle_joint</joint_name>
@@ -149,4 +150,17 @@
         </visual>
     </link>
+    <link name="livox_lidar_link">
+        <visual>
+            <geometry>
+                <mesh filename="file:///home/sohithvulipe/ws_livox/src/PB_RMSimulation/src/rm_simulation/pb_rm_simulation/meshes/mid360.stl" scale="0.0008 0.0008 0.0008" />
+            </geometry>
+        </visual>
+    </link>
+    <!-- Attach the LiDAR link to the base_link -->
+    <joint name="livox_lidar_joint" type="fixed">
+        <parent link="base_link"/>
+        <child link="livox_lidar_link"/>
+        <origin xyz="0.3 0 0.5" rpy="1.57 3.14 0" />  <!-- Adjust position and orientation as needed -->
+    </joint>
     <gazebo reference="base_link">
         <material>Gazebo/Orange</material>
@@ -165,8 +179,8 @@
         <origin xyz="0.17 0 0.005" rpy="0 0 0"/>
     </xacro:sensor_hokuyo>
-    <xacro:include filename="$(find ros2_livox_simulation)/urdf/mid360.xacro"/>
+    <!-- <xacro:include filename="$(find ros2_livox_simulation)/urdf/mid360.xacro"/>
 <xacro:mid360 parent="base_link" name="livox_lidar" topic="/livox/lidar">
-  <origin xyz="0.3 0 0.5" rpy="0 3.14 0" />
-</xacro:mid360>
+  <origin xyz="0 0 0" rpy="0 0 0" />
+</xacro:mid360> -->
     <xacro:sensor_imu prefix="imu" parent="base_link">
         <!-- <origin xyz="-0.32 0 0.05" rpy="0 0.5 0"/> -->
@@ -177,8 +191,9 @@
         <!-- <origin xyz="0.212 0 0.065" rpy="0 0 0"/> -->
     </xacro:sensor_asus_xtion>
-    <xacro:sensor_asus_xtion2 prefix="camera2" parent="base_link">
-        <origin xyz="0.215 0 5" rpy="0 1.57 0"/>
+    <!-- <xacro:sensor_asus_xtion2 prefix="camera2" parent="base_link">
+        <origin xyz="0.215 0 5" rpy="0 1.57 0"/> -->
         <!-- <origin xyz="0.212 0 0.065" rpy="0 0 0"/> -->
-    </xacro:sensor_asus_xtion2>
+    <!-- </xacro:sensor_asus_xtion2> -->
+    <!-- <xacro:sensor_light prefix="light1" parent="base_link"/> -->
     <!-- wheels -->
     <xacro:corner_link lon_label="front" lat_label="left" reflect="1"/>

File: rover_description/urdf/sensors/all_sensors.urdf.xacro (robot description, xacro)
@@ -24,4 +24,5 @@
   <!-- Hokuyo -->
   <xacro:include filename="$(find rover_description)/urdf/sensors/asus_xtion.urdf.xacro" />
-  <xacro:include filename="$(find rover_description)/urdf/sensors/asus_xtion2.urdf.xacro" />
+  <!-- <xacro:include filename="$(find rover_description)/urdf/sensors/asus_xtion2.urdf.xacro" />  -->
+  <!-- <xacro:include filename="$(find rover_description)/urdf/sensors/light.urdf.xacro" />  -->
 </robot>
